File: kicad/template.kicad_sch (KiCad schematic)
At the start: 7 parts, among them J1 Bus_PCI_Express_x1, J6 USB_C_Receptacle_USB2.0_16P, U1 MCP25625T-E/ML, U2 RP2040, U4 W25Q128JVP, X1 ABM8-272-T3, Y1 X322516MLB4SI

Commit message: init cihad's status module
Parts:
- removed U1: MCP25625T-E/ML, challenge_template:QFN28_6X6MC_MCH, symbol challenge symbols:MCP25625T-E_ML
- removed X1: ABM8-272-T3, challenge_template:ABM8-272-T3_ABR, symbol challenge symbols:ABM8-272-T3
- removed Y1: X322516MLB4SI, challenge_template:OSC_X322516MLB4SI, symbol challenge symbols:X322516MLB4SI
- added C1, C10, C11, C16, C17, C18, C19, C2, C4, C6, C7, C8, C9: 100n, Capacitor_SMD:C_0402_1005Metric, symbol Device:C
- added C12, C13: 22p, Capacitor_SMD:C_0402_1005Metric, symbol Device:C
- added C14, C15: 15p, Capacitor_SMD:C_0402_1005Metric, symbol Device:C
- added C3, C5: 1u, Capacitor_SMD:C_0402_1005Metric, symbol Device:C
- added R1, R2: 27, Resistor_SMD:R_0402_1005Metric, symbol Device:R
- added R3, R4: 5.1k, Resistor_SMD:R_0402_1005Metric, symbol Device:R
- added R5, R6: 1k, Resistor_SMD:R_0402_1005Metric, symbol Device:R
- added S1: TS-1187A-B-A-B, TS-1187A-B-A-B:SW_TS-1187A-B-A-B, symbol TS-1187A-B-A-B:TS-1187A-B-A-B
- added U9: MCP25625T-E/ML, MCP25625T_E_ML:QFN28_6X6MC_MCH, symbol MCP25625:MCP25625T-E_ML
- added X2: ABM8-272-T3, ABM8-272-T3:ABM8-272-T3_ABR, symbol crystal:ABM8-272-T3
- added Y1: X322516MLB4SI, X322516MLB4SI:OSC_X322516MLB4SI, symbol X322516MLB4SI:X322516MLB4SI
Connections:
- net +3.3V: now also U4.8 (VCC), C16.1
- net +5V: now also C17.1, U9.19 (VDDA)
- net GND: now also U2.19 (TESTEN), U2.57 (GND), C1.2, C10.2, C11.2, C12.2, C13.2, C14.2, C15.2, C16.2, C17.2, C18.2, C19.1, C2.2, C3.2, C4.2, C5.2, C6.2, C7.2, C8.2, C9.2, R3.1, R4.2, S1.A, S1.B, X2.2, X2.4, Y1.2, Y1.4
- net QSPI_SS: now reaches U4.1 (~{CS})
- net QSPI_SS: now also U2.56 (QSPI_SS), R6.1
- net QSPI_SD1: now reaches U4.2 (DO(IO1))
- net QSPI_SD1: now also U2.55 (QSPI_SD1)
- net QSPI_SD2: now reaches U4.3 (IO2)
- net QSPI_SD2: now also U2.54 (QSPI_SD2)
- net QSPI_SD0: now reaches U4.5 (DI(IO0))
- net QSPI_SD0: now also U2.53 (QSPI_SD0)
- net QSPI_SCLK: now reaches U4.6 (CLK)
- net QSPI_SCLK: now also U2.52 (QSPI_SCLK)
- net QSPI_SD3: now reaches U4.7 (IO3)
- net QSPI_SD3: now also U2.51 (QSPI_SD3)
- net +3V3: now reaches U2.1 (IOVDD), U2.10 (IOVDD), U2.22 (IOVDD), U2.33 (IOVDD), U2.42 (IOVDD), U2.49 (IOVDD)
- net +3V3: now also U2.43 (ADC_AVDD), U2.44 (VREG_IN), U2.48 (USB_VDD), C10.1, C11.1, C18.1, C19.2, C4.1, C5.1, C6.1, C7.1, C8.1, C9.1, U9.11 (VIO), U9.3 (VDD)
- net XIN: now reaches U2.20 (XIN)
- net XIN: now also C14.1, X2.1
- net XOUT: now reaches U2.21 (XOUT)
- net XOUT: now also R5.1
- net +1V1: now reaches U2.23 (DVDD), U2.50 (DVDD)
- net +1V1: now also U2.45 (VREG_VOUT), C1.1, C2.1, C3.1
- net SWCLK: now reaches U2.24 (SWCLK)
- net SWD: now reaches U2.25 (SWD)
- net INT: now reaches U2.39 (GPIO27_ADC1)
- net SDA: now reaches U2.40 (GPIO28_ADC2)
- net SCL: now reaches U2.41 (GPIO29_ADC3)
- net USB_D2-: now reaches U2.46 (USB_DM)
- net USB_D2-: now also R2.2
- net USB_D2+: now reaches U2.47 (USB_DP)
- net USB_D2+: now also R1.2
- net at J6.A5 (CC1): now also R3.2
- net USB_D+: now reaches J6.A6 (D+), J6.B6 (D+)
- net USB_D+: now also R1.1
- net USB_D-: now reaches J6.A7 (D-), J6.B7 (D-)
- net USB_D-: now also R2.1
- net at J6.B5 (CC2): now also R4.1
- new net OSC1: C13.1, U9.21 (OSC1), Y1.3
- new net OSC2: C12.1, U9.20 (OSC2), Y1.1
- new net XOUT_pre: C15.1, R5.2, X2.3
- new net rx(CAN): U9.10 (RXD), U9.5 (RXCAN)
- new net tx(CAN): U9.16 (TXD), U9.4 (TXCAN)
- new net ~{USB_BOOT_S}: R6.2, S1.C, S1.D
- no-connect marks 8 -> 9
Other:
- note added: "Make sure C10 is close to pin 44 of RP2040"
- note added: "Make sure C8 is close to pin 45 of RP2040"
- note added: "Make sure R3 and R4 are close to RP2040"
- note removed: "CAN Crystal"
